Commit message: Repair the physical model
Repair physical parameter model and geometric model separation problem. A line command was added to the "collision" of the "define_link" of the macro module. This command sets the origin of the physical model initialization (not just the beginning of the geometric model setting).

File: mentorRobot_clean.xacro (robot description, xacro)
@@ -76,4 +76,5 @@
 					<mesh filename = "${model_dae}"/>
 				</geometry>
+                                <origin xyz = "${model_xyz}" rpy = "0 0 0"/>
 			</collision>
 			<inertial>

Commit message: Add a Laser and two cameras.
Add a Laser and two cameras, and include a robot.gazebo document for description their parameters.

File: mentorRobot_clean.xacro (robot description, xacro)
@@ -25,4 +25,21 @@
         <xacro:property name = "neck_position" value = "0 0 0.33506"/>
         <xacro:property name = "neck_axis" value = "0 0 1"/>
+        <xacro:property name = "laser_data" value = "package://urdf_tutorial/meshes/3DLaser.DAE"/>
+        <xacro:property name = "laser_xyz" value = "-0.513063 0 -0.557158"/>
+        <xacro:property name = "laser_mess" value = "1e-5"/>
+        <xacro:property name = "laser_ixx" value = "1e-6"/>   <xacro:property name = "laser_izz" value = "1e-6"/>
+        <xacro:property name = "laser_ixz" value = "0"/>        <xacro:property name = "laser_iyz" value = "0"/>
+        <xacro:property name = "laser_ixy" value = "0"/>        <xacro:property name = "laser_iyy" value = "1e-6"/>
+        <xacro:property name = "laser_position" value = "0.513063 0 0.557158"/>
+        <xacro:property name = "right_eye_data" value = "package://urdf_tutorial/meshes/RightEye.DAE"/>
+        <xacro:property name = "left_eye_data" value = "package://urdf_tutorial/meshes/LeftEye.DAE"/>
+        <xacro:property name = "right_eye_xyz" value = "-0.0906 -0.4 -0.771774"/>
+        <xacro:property name = "left_eye_xyz" value = "-0.0906 0.4 -0.771774"/>
+        <xacro:property name = "eye_mess" value = "1e-5"/>
+        <xacro:property name = "eye_ixx" value = "1e-6"/>   <xacro:property name = "eye_izz" value = "1e-6"/>
+        <xacro:property name = "eye_ixz" value = "0"/>        <xacro:property name = "eye_iyz" value = "0"/>
+        <xacro:property name = "eye_ixy" value = "0"/>        <xacro:property name = "eye_iyy" value = "1e-6"/>
+        <xacro:property name = "right_eye_position" value = "0.0906 0.4 0.243388"/>
+        <xacro:property name = "left_eye_position" value = "0.0906 -0.4 0.243388"/>
         <xacro:property name = "rh_leg_data" value = "package://urdf_tutorial/meshes/WheelTuR.DAE"/>
         <xacro:property name = "rb_leg_data" value = "package://urdf_tutorial/meshes/WheelTuR2.DAE"/>
@@ -101,6 +118,14 @@
                 </joint>
         </xacro:macro>
+        <xacro:macro name = "define_fixed_joint" params = "name type parent child position">
+                <joint name = "${name}" type = "${type}">
+                        <parent link = "${parent}"/>
+                        <child link = "${child}"/>
+                        <origin xyz = "${position}"/>
+                </joint>
+        </xacro:macro>
 <!--Useing-->
 <!--================================Instaniation==========================================================-->
+	<xacro:include filename = "$(find urdf_tutorial)/urdf/robot.gazebo"/>
 	<xacro:define_link name = "body" model_dae = "${body_data}" model_xyz = "${body_xyz}" model_mess = "${body_mess}">
 		<inertia ixx =  "${body_ixx}" ixz = "${body_ixz}" ixy = "${body_ixy}" izz = "${body_izz}" iyz = "${body_iyz}" iyy = "${body_iyy}"/>
@@ -116,4 +141,16 @@
                 <limit effort = "1000" lower = "-1.571" upper = "1.571" velocity = "0.5"/>
         </xacro:define_limit_joint>
+        <xacro:define_link name = "hokuyo_link" model_dae = "${laser_data}" model_xyz = "${laser_xyz}" model_mess = "${laser_mess}">
+                <inertia ixx =  "${laser_ixx}" ixz = "${laser_ixz}" ixy = "${laser_ixy}" izz = "${laser_izz}" iyz = "${laser_iyz}" iyy = "${laser_iyy}"/>
+        </xacro:define_link>
+        <xacro:define_fixed_joint name = "Laserfixed" type = "fixed" parent = "body" child = "hokuyo_link" position ="${laser_position}"/>
+        <xacro:define_link name = "camera1_link" model_dae = "${right_eye_data}" model_xyz = "${right_eye_xyz}" model_mess = "${eye_mess}">
+                <inertia ixx =  "${eye_ixx}" ixz = "${eye_ixz}" ixy = "${eye_ixy}" izz = "${eye_izz}" iyz = "${eye_iyz}" iyy = "${eye_iyy}"/>
+        </xacro:define_link>
+        <xacro:define_fixed_joint name = "RightEyefixed" type = "fixed" parent = "camera" child = "camera1_link" position ="${right_eye_position}"/>
+        <xacro:define_link name = "camera2_link" model_dae = "${left_eye_data}" model_xyz = "${left_eye_xyz}" model_mess = "${eye_mess}">
+                <inertia ixx =  "${eye_ixx}" ixz = "${eye_ixz}" ixy = "${eye_ixy}" izz = "${eye_izz}" iyz = "${eye_iyz}" iyy = "${eye_iyy}"/>
+        </xacro:define_link>
+        <xacro:define_fixed_joint name = "LeftEyefixed" type = "fixed" parent = "camera" child = "camera2_link" position ="${left_eye_position}"/>
 	<xacro:define_link name = "rh_leg" model_dae = "${rh_leg_data}" model_xyz = "${rh_leg_xyz}" model_mess = "${leg_mess}">
                 <inertia ixx =  "${leg_ixx}" ixz = "${leg_ixz}" ixy = "${leg_ixy}" izz = "${leg_izz}" iyz = "${leg_iyz}" iyy = "${leg_iyy}"/>
